File: ProPrj_FaultMonitor_2025-11-15(4)/ProPrj_FaultMonitor_2025-11-15(4).kicad_sch (KiCad schematic)
At the start: 16 parts, among them CN1 XH-2A, CN2 ZX-XH2.54-6PZZ, CN3 ZX-XH2.54-3PZZ, CN4 XH-2A, U2 DS18B20T(XBLW), U3 ESP32-DevKitC

Commit message: minor edits
Parts:
- removed ?: (no value), ProPrj_Fau-easyedapro:, symbol ProPrj_Fau-easyedapro:Drawing-Symbol_A4
- removed LED6, LED7, LED8, LED9: DY-333SDRD-SN-A3(EL)(HF), ProPrj_Fau-easyedapro:ED-TH_BD5.8-P2.54-R-FD, symbol ProPrj_Fau-easyedapro:EL504RD
- removed R1, R2, R3, R4: 2.2kΩ, ProPrj_Fau-easyedapro:R0603, symbol ProPrj_Fau-easyedapro:Res
- added D1, D2, D3, D4: LED, symbol Device:LED
- added R1, R2, R3, R4: R, symbol Device:R
- renumbered CN1 to 24V, CN3 to 24V, CN4 to 5V, CN2 to IO
Connections:
- net GND: now also D1.1 (K), D2.1 (K), D3.1 (K), D4.1 (K)
- net at U3.8 (IO33): now also R3.1
- net at U3.7 (IO32): now also R4.1
- net at U3.10 (IO26): now also R1.1
- net at U3.9 (IO25): now also R2.1
- net CURR_SENS: no longer names the net of 24V.3, U3.12 (IO14)
- new net: D2.2 (A), R2.2
- new net: D4.2 (A), R4.2
- new net: D3.2 (A), R3.2
- new net: D1.2 (A), R1.2

Commit message: minor formatting changes
Parts:
- renumbered U3 to U1
Connections:
- net GND: now also U1.14 (GND)
Changed lines of the file:
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@@
 		(color 0 0 0 0)
 	)
+	(junction
+		(at 17.78 43.18)
+		(diameter 0)
+		(color 0 0 0 0)
+	)
 	(wire
 		(pts
@@
 	(wire
 		(pts
+			(xy 17.78 45.72) (xy 17.78 43.18)
+		)
+		(stroke
+			(width 0)
+			(type default)
+		)
+	)
+	(wire
+		(pts
 			(xy 40.64 20.32) (xy 50.8 20.32)
 		)
@@
 		(pts
 			(xy 29.21 109.22) (xy 40.64 109.22)
+		)
+		(stroke
+			(width 0)
+			(type default)
+		)
+	)
+	(wire
+		(pts
+			(xy 17.78 43.18) (xy 50.8 43.18)
 		)
 		(stroke
@@
 		)
 		(property "Value" "GND"
-			(at 80.01 10.16 90)
+			(at 81.28 10.16 90)
 			(effects
 				(font
@@
 	(symbol
 		(lib_id "ProPrj_Fau-easyedapro:Ground-GND")
-		(at 17.78 43.18 0)
+		(at 17.78 45.72 0)
 		(unit 1)
 		(exclude_from_sim no)
@@
 		(dnp no)
 		(property "Reference" "#PWR?"
-			(at 17.78 43.18 0)
+			(at 17.78 45.72 0)
 			(effects
 				(font
@@
 		)
 		(property "Value" "GND"
-			(at 17.78 49.53 0)
+			(at 17.78 52.07 0)
 			(effects
 				(font
@@
 		)
 		(property "Footprint" "ProPrj_Fau-easyedapro:"
-			(at 17.78 43.18 0)
+			(at 17.78 45.72 0)
 			(effects
 				(font
@@
 		)
 		(property "Datasheet" ""
-			(at 17.78 43.18 0)
+			(at 17.78 45.72 0)
 			(effects
 				(font
@@
 		)
 		(property "Description" ""
-			(at 17.78 43.18 0)
+			(at 17.78 45.72 0)
 			(effects
 				(font
@@
 		(on_board yes)
 		(dnp no)
-		(property "Reference" "U3"
-			(at 53.34 7.62 0)
+		(property "Reference" "U1"
+			(at 61.976 6.096 0)
 			(effects
 				(font
@@
 		)
 		(property "Value" "ESP32-DevKitC"
-			(at 53.34 60.96 0)
+			(at 62.23 60.452 0)
 			(effects
 				(font
@@
 			(project ""
 				(path "/64884559-cbe4-442b-837a-f1967fbf7136"
-					(reference "U3")
+					(reference "U1")
 					(unit 1)
 				)
