File: fault-monitor/fault-monitor/fault-monitor.kicad_sch (KiCad schematic)
At the start: 21 parts, among them J1 Conn_01x03, J2 Conn_01x06, J3 Conn_01x02, J4 Conn_01x02, J5 Conn_01x02, J6 Conn_01x02, J7 Conn_01x06, U1 ESP32-DevKitC

Commit message: full redo of pcb cuz we fucked up the usb port
Parts:
- J1: footprint TerminalBlock_WAGO_3D:TerminalBlock_WAGO_2601-1103_1x03_P3.50mm_Horizontal-3D -> TerminalBlock:TerminalBlock_MaiXu_MX126-5.0-03P_1x03_P5.00mm
- J2, J7: footprint TerminalBlock_WAGO_3D:TerminalBlock_WAGO_2601-1106_1x06_P3.50mm_Horizontal-3D -> TerminalBlock:TerminalBlock_MaiXu_MX126-5.0-06P_1x06_P5.00mm
- J3, J4, J6: footprint TerminalBlock_WAGO_3D:TerminalBlock_WAGO_2601-1102_1x02_P3.50mm_Horizontal-3D -> TerminalBlock:TerminalBlock_MaiXu_MX126-5.0-02P_1x02_P5.00mm
Changed lines of the file:
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@@
 			)
 		)
-		(property "Footprint" "TerminalBlock_WAGO_3D:TerminalBlock_WAGO_2601-1106_1x06_P3.50mm_Horizontal-3D"
+		(property "Footprint" "TerminalBlock:TerminalBlock_MaiXu_MX126-5.0-06P_1x06_P5.00mm"
 			(at 124.46 130.81 0)
 			(effects
@@
 			)
 		)
-		(property "Footprint" "TerminalBlock_WAGO_3D:TerminalBlock_WAGO_2601-1102_1x02_P3.50mm_Horizontal-3D"
+		(property "Footprint" "TerminalBlock:TerminalBlock_MaiXu_MX126-5.0-02P_1x02_P5.00mm"
 			(at 124.46 110.49 0)
 			(effects
@@
 			)
 		)
-		(property "Footprint" "TerminalBlock_WAGO_3D:TerminalBlock_WAGO_2601-1102_1x02_P3.50mm_Horizontal-3D"
+		(property "Footprint" "TerminalBlock:TerminalBlock_MaiXu_MX126-5.0-02P_1x02_P5.00mm"
 			(at 106.68 17.78 0)
 			(effects
@@
 			)
 		)
-		(property "Footprint" "TerminalBlock_WAGO_3D:TerminalBlock_WAGO_2601-1102_1x02_P3.50mm_Horizontal-3D"
+		(property "Footprint" "TerminalBlock:TerminalBlock_MaiXu_MX126-5.0-02P_1x02_P5.00mm"
 			(at 121.92 38.1 0)
 			(effects
@@
 			)
 		)
-		(property "Footprint" "TerminalBlock_WAGO_3D:TerminalBlock_WAGO_2601-1103_1x03_P3.50mm_Horizontal-3D"
+		(property "Footprint" "TerminalBlock:TerminalBlock_MaiXu_MX126-5.0-03P_1x03_P5.00mm"
 			(at 26.67 58.42 0)
 			(effects
@@
 			)
 		)
-		(property "Footprint" "TerminalBlock_WAGO_3D:TerminalBlock_WAGO_2601-1106_1x06_P3.50mm_Horizontal-3D"
+		(property "Footprint" "TerminalBlock:TerminalBlock_MaiXu_MX126-5.0-06P_1x06_P5.00mm"
 			(at 124.46 91.44 0)
 			(effects
