Commit message: Fix camera in sim

File: description/rover_model/urdf/plugins.ignition.xacro (robot description, xacro)
@@ -232,5 +232,5 @@
                     <clip>
                         <near>0.3</near>
-                        <far>10</far>
+                        <far>300</far>
                     </clip>
                 </depth_camera>

File: description/rover_model/urdf/stand_link.urdf.xacro (robot description, xacro)
@@ -88,5 +88,5 @@
         <parent link="zed_link"/>
         <child link="left_camera_link"/>
-        <origin xyz="0 ${ZED_stereo_offset / 2.0} 0" rpy="0 0 0"/>
+        <origin xyz="0.00001 ${ZED_stereo_offset / 2.0} 0" rpy="0 0 0"/>
     </joint>
     <!-- Generate an optical frame http://www.ros.org/reps/rep-0103.html#suffix-frames so that ros and opencv can operate on the camera frame correctly -->
