Commit message: oisjgv

File: description/rover_model/urdf/wheels.urdf.xacro (robot description, xacro)
@@ -30,5 +30,5 @@
             <origin xyz="0 0 0" rpy="0 0 0" />
             <geometry>
-                <mesh filename="package://description/rover_model/meshes/leftwheel_link.STL" />
+                <mesh filename="package://description/rover_model/meshes/left_wheel_link.STL" />
             </geometry>
             <material name="">
@@ -39,5 +39,5 @@
             <origin xyz="0 0 0" rpy="0 0 0" />
             <geometry>
-                <mesh filename="package://description/rover_model/meshes/leftwheel_link.STL" />
+                <mesh filename="package://description/rover_model/meshes/left_wheel_link.STL" />
             </geometry>
         </collision> -->
@@ -79,5 +79,5 @@
             <origin xyz="0 0 0" rpy="0 0 0" />
             <geometry>
-                <mesh filename="package://description/rover_model/meshes/rightwheel_link.STL" />
+                <mesh filename="package://description/rover_model/meshes/right_wheel_link.STL" />
             </geometry>
             <material name="">
