Commit message: fixed filenames of wheels and lidars

File: description/rover_model/urdf/timbot.urdf.xacro (robot description, xacro)
@@ -83,5 +83,5 @@
 			<origin xyz="0 0 0" rpy="0 0 0" />
 			<geometry>
-				<mesh filename="package://description/rover_model/meshes/lidar_link.STL" />
+				<mesh filename="package://description/rover_model/meshes/top_lidar_link.STL" />
 			</geometry>
 			<material name="">
@@ -122,5 +122,5 @@
 			<origin xyz="0 0 0" rpy="0 0 0" />
 			<geometry>
-				<mesh filename="package://description/rover_model/meshes/lidar_link.STL" />
+				<mesh filename="package://description/rover_model/meshes/bottom_lidar_link.STL" />
 			</geometry>
 			<material name="">

Commit message: filename fix #2

File: description/rover_model/urdf/timbot.urdf.xacro (robot description, xacro)
@@ -92,5 +92,5 @@
 			<origin xyz="0 0 0" rpy="0 0 0" />
 			<geometry>
-				<mesh filename="package://description/rover_model/meshes/lidar_link.STL" />
+				<mesh filename="package://description/rover_model/meshes/top_lidar_link.STL" />
 			</geometry>
 		</collision>
@@ -131,5 +131,5 @@
 			<origin xyz="0 0 0" rpy="0 0 0" />
 			<geometry>
-				<mesh filename="package://description/rover_model/meshes/lidar_link.STL" />
+				<mesh filename="package://description/rover_model/meshes/bottom_lidar_link.STL" />
 			</geometry>
 		</collision>

File: description/rover_model/urdf/wheels.urdf.xacro (robot description, xacro)
@@ -88,5 +88,5 @@
             <origin xyz="0 0 0" rpy="0 0 0" />
             <geometry>
-                <mesh filename="package://description/rover_model/meshes/rightwheel_link.STL" />
+                <mesh filename="package://description/rover_model/meshes/right_wheel_link.STL" />
             </geometry>
         </collision> -->
