Commit message: Fix robot not moving in sim
Wheels seem to be unable to touch the ground due to chassis_link size changed in e8c66e9

File: description/rover_model/urdf/timbot.urdf.xacro (robot description, xacro)
@@ -26,5 +26,5 @@
 	<link name="chassis_link">
 		<inertial>
-			<origin xyz="-0.040859 0.00033673 10.54592" rpy="0 0 0" />
+			<origin xyz="-0.040859 0.00033673 -0.054592" rpy="0 0 0" />
 			<mass value="40.135" />
 			<inertia
@@ -54,5 +54,5 @@
 			<origin xyz="0 0 0" rpy="0 0 0" />
 			<geometry>
-				<box size="0.9 0.6 0.3"/>
+				<box size="0.9 0.6 0.2"/>
 			</geometry>
 		</collision>
