Commit message: imu position patch

File: description/rover_model/urdf/stand_link.urdf.xacro (robot description, xacro)
@@ -112,5 +112,5 @@
         </inertial>
         <visual>
-            <origin xyz="0 0 0.61854" rpy="0 0 0" /> <!-- Physical imu located on stand -->
+            <origin xyz="0 0 0" rpy="0 0 0" /> <!-- Physical imu located on stand -->
             <!-- z-pos of visual model moved back up to stand height
                  z: imu_z_dist_to_stand + chassis_to_stand_link_z_dist + chassis_to_base_link_dist} -->
@@ -123,5 +123,5 @@
         </visual>
         <collision>
-            <origin xyz="0 0 0.61854" rpy="0 0 0" />
+            <origin xyz="0 0 0" rpy="0 0 0" />
             <geometry>
                 <mesh filename="package://description/rover_model/meshes/imu_link.STL" />

Commit message: got claude to fix the values

File: description/rover_model/urdf/stand_link.urdf.xacro (robot description, xacro)
@@ -35,5 +35,5 @@
     </link>
     <joint name="stand_joint" type="fixed">
-        <origin xyz="0.178 0.001524 0.26861" rpy="0 0 0" />
+        <origin xyz="-0.1268 -0.0003302 0.6548" rpy="0 0 0" />
         <parent link="chassis_link" />
         <child link="stand_link" />
@@ -74,5 +74,5 @@
     </link>
     <joint name="zed_joint" type="fixed">
-        <origin xyz="0.044163 0 ${ZED_camera_to_top_plate_z}" rpy="0 ${ZED_camera_pitch} 0" />
+        <origin xyz="0.073649 0 0.10196" rpy="0 0.21468 0" />
         <parent link="stand_link" />
         <child link="zed_link" />
@@ -130,5 +130,5 @@
     </link>
     <joint name="imu_joint" type="fixed">
-        <origin xyz="0.159347 0 0" rpy="0 0 0" />
+        <origin xyz="0.096934 0.026936 0.0022059" rpy="0 0 0" />
         <!-- The x-pos is same as it's actual position on the stand, but z-pos same as base_link
              x: imu_x_dist_to_stand + chassis_to_stand_link_x_dist -->
@@ -170,8 +170,8 @@
     </link>
     <joint name="gps_joint" type="fixed">
-        <origin xyz="-0.054799 0 0.0095015" rpy="0 0 0" />
+        <origin xyz="-0.028849 -0.027397 0.009525" rpy="0 0 0" />
         <parent link="stand_link" />
         <child link="gps_link" />
-        <axis xyz="0 0 1" />
+        <axis xyz="0 0 0" />
     </joint>
     <gazebo reference="gps_link">

File: description/rover_model/urdf/timbot.urdf.xacro (robot description, xacro)
@@ -59,5 +59,5 @@
 	</link>
 	<joint name="chassis_joint" type="fixed">
-		<origin xyz="0 0 0.34041" rpy="0 0 0" />
+		<origin xyz="0.257302 0 0.130140280102375" rpy="0 0 0" />
 		<parent link="base_link" />
 		<child link="chassis_link" />
@@ -97,5 +97,5 @@
 	</link>
 	<joint name="top_lidar_joint" type="fixed">
-		<origin xyz="0.52049 -0.005698 ${distance_to_second_lidar - 0.069334}" rpy="0 0 0" />
+		<origin xyz="0.20922 -0.00047545 0.34705" rpy="0 0 0" />
 		<!-- before z =  0.0056661 -->
 		<parent link="chassis_link" />
@@ -136,5 +136,5 @@
 	</link>
 	<joint name="bottom_lidar_joint" type="fixed">
-		<origin xyz="0.52049 -0.005698 -0.069334" rpy="0 0 0" />
+		<origin xyz="0.20871 -1.6731E-05 0.14385" rpy="0 0 0" />
 		<parent link="chassis_link" />
 		<child link="bottom_lidar_link" />

File: description/rover_model/urdf/wheels.urdf.xacro (robot description, xacro)
@@ -49,8 +49,8 @@
     </link>
     <joint name="left_wheel_joint" type="continuous">
-        <origin xyz="0.30478 0.40518 -0.21541" rpy="0 0 0" />
+        <origin xyz="0 0.337221649344587 0" rpy="0 0 0" />
         <parent link="chassis_link" />
         <child link="left_wheel_link" />
-        <axis xyz="0 1 0" />
+        <axis xyz="0 -1 0" />
         <limit effort="100.0" velocity="20.0"/>
     </joint>
@@ -98,8 +98,8 @@
     </link>
     <joint name="right_wheel_joint" type="continuous">
-        <origin xyz="0.30482 -0.40518 -0.21541" rpy="0 0 0" />
+        <origin xyz="0 -0.337221649344586 0" rpy="0 0 0" />
         <parent link="chassis_link" />
         <child link="right_wheel_link" />
-        <axis xyz="0 1 0" />
+        <axis xyz="0 -1 0" />
         <limit effort="100.0" velocity="20.0"/>
     </joint>
@@ -142,5 +142,5 @@
     </link>
     <joint name="caster_joint" type="fixed">
-        <origin xyz="-0.36833 0.001524 -0.13183" rpy="0 0 0" />
+        <origin xyz="-0.67301 7.5398E-05 0.070217" rpy="0 0 0" />
         <parent link="chassis_link" />
         <child link="caster_link" />

Commit message: display launch patch to remove refs to espresso

File: description/rover_model/urdf/stand_link.urdf.xacro (robot description, xacro)
@@ -35,5 +35,5 @@
     </link>
     <joint name="stand_joint" type="fixed">
-        <origin xyz="-0.1268 -0.0003302 0.6548" rpy="0 0 0" />
+        <origin xyz="0.178 0.001524 0.26861" rpy="0 0 0" />
         <parent link="chassis_link" />
         <child link="stand_link" />
@@ -74,5 +74,5 @@
     </link>
     <joint name="zed_joint" type="fixed">
-        <origin xyz="0.073649 0 0.10196" rpy="0 0.21468 0" />
+        <origin xyz="0.044163 0 ${ZED_camera_to_top_plate_z}" rpy="0 ${ZED_camera_pitch} 0" />
         <parent link="stand_link" />
         <child link="zed_link" />
@@ -130,5 +130,5 @@
     </link>
     <joint name="imu_joint" type="fixed">
-        <origin xyz="0.096934 0.026936 0.0022059" rpy="0 0 0" />
+        <origin xyz="0.159347 0 0" rpy="0 0 0" />
         <!-- The x-pos is same as it's actual position on the stand, but z-pos same as base_link
              x: imu_x_dist_to_stand + chassis_to_stand_link_x_dist -->
@@ -170,8 +170,8 @@
     </link>
     <joint name="gps_joint" type="fixed">
-        <origin xyz="-0.028849 -0.027397 0.009525" rpy="0 0 0" />
+        <origin xyz="-0.054799 0 0.0095015" rpy="0 0 0" />
         <parent link="stand_link" />
         <child link="gps_link" />
-        <axis xyz="0 0 0" />
+        <axis xyz="0 0 1" />
     </joint>
     <gazebo reference="gps_link">

File: description/rover_model/urdf/timbot.urdf.xacro (robot description, xacro)
@@ -59,5 +59,5 @@
 	</link>
 	<joint name="chassis_joint" type="fixed">
-		<origin xyz="0.257302 0 0.130140280102375" rpy="0 0 0" />
+		<origin xyz="0 0 0.34041" rpy="0 0 0" />
 		<parent link="base_link" />
 		<child link="chassis_link" />
@@ -97,5 +97,5 @@
 	</link>
 	<joint name="top_lidar_joint" type="fixed">
-		<origin xyz="0.20922 -0.00047545 0.34705" rpy="0 0 0" />
+		<origin xyz="0.52049 -0.005698 ${distance_to_second_lidar - 0.069334}" rpy="0 0 0" />
 		<!-- before z =  0.0056661 -->
 		<parent link="chassis_link" />
@@ -136,5 +136,5 @@
 	</link>
 	<joint name="bottom_lidar_joint" type="fixed">
-		<origin xyz="0.20871 -1.6731E-05 0.14385" rpy="0 0 0" />
+		<origin xyz="0.52049 -0.005698 -0.069334" rpy="0 0 0" />
 		<parent link="chassis_link" />
 		<child link="bottom_lidar_link" />

File: description/rover_model/urdf/wheels.urdf.xacro (robot description, xacro)
@@ -49,8 +49,8 @@
     </link>
     <joint name="left_wheel_joint" type="continuous">
-        <origin xyz="0 0.337221649344587 0" rpy="0 0 0" />
+        <origin xyz="0.30478 0.40518 -0.21541" rpy="0 0 0" />
         <parent link="chassis_link" />
         <child link="left_wheel_link" />
-        <axis xyz="0 -1 0" />
+        <axis xyz="0 1 0" />
         <limit effort="100.0" velocity="20.0"/>
     </joint>
@@ -98,8 +98,8 @@
     </link>
     <joint name="right_wheel_joint" type="continuous">
-        <origin xyz="0 -0.337221649344586 0" rpy="0 0 0" />
+        <origin xyz="0.30482 -0.40518 -0.21541" rpy="0 0 0" />
         <parent link="chassis_link" />
         <child link="right_wheel_link" />
-        <axis xyz="0 -1 0" />
+        <axis xyz="0 1 0" />
         <limit effort="100.0" velocity="20.0"/>
     </joint>
@@ -142,5 +142,5 @@
     </link>
     <joint name="caster_joint" type="fixed">
-        <origin xyz="-0.67301 7.5398E-05 0.070217" rpy="0 0 0" />
+        <origin xyz="-0.36833 0.001524 -0.13183" rpy="0 0 0" />
         <parent link="chassis_link" />
         <child link="caster_link" />

Commit message: setting up the ENU for magnometer

File: description/rover_model/urdf/stand_link.urdf.xacro (robot description, xacro)
@@ -101,5 +101,5 @@
     <link name="imu_link">
         <inertial>
-            <origin xyz="3.0642E-07 -2.658E-07 0.0062442" rpy="3.14159 0 0" />
+            <origin xyz="3.0642E-07 -2.658E-07 0.0062442" rpy="0 0 0" />
             <mass value="0.016518" />
             <inertia
@@ -112,5 +112,5 @@
         </inertial>
         <visual>
-            <origin xyz="0 0 0" rpy="3.14159 0 0" /> <!-- Physical imu located on stand -->
+            <origin xyz="0 0 0" rpy="0 0 0" /> <!-- mesh origin matches FLU imu_link frame -->
             <!-- z-pos of visual model moved back up to stand height
                  z: imu_z_dist_to_stand + chassis_to_stand_link_z_dist + chassis_to_base_link_dist} -->
@@ -123,5 +123,5 @@
         </visual>
         <collision>
-            <origin xyz="0 0 0" rpy="3.14159 0 0" />
+            <origin xyz="0 0 0" rpy="0 0 0" />
             <geometry>
                 <mesh filename="package://description/rover_model/meshes/imu_link.STL" />
@@ -130,5 +130,10 @@
     </link>
     <joint name="imu_joint" type="fixed">
-        <origin xyz="0.0969 0.0229 0" rpy="3.14159 0 0" />
+        <!-- imu_link is FLU (x-forward, y-left, z-up), aligned with base_link.
+             ⚠ This rpy MUST match the PHYSICAL sensor axes. It is only valid if the
+             IMU is physically mounted FLU. If the chip is mounted flipped, TF will
+             rotate gyro/accel 180° about X (inverting roll/pitch and FLIPPING yaw
+             sign in ekf_local). Verify on the bench (see notes) before trusting. -->
+        <origin xyz="0.0969 0.0229 0" rpy="0 0 0" />
         <!-- The x-pos is same as it's actual position on the stand, but z-pos same as base_link
              x: imu_x_dist_to_stand + chassis_to_stand_link_x_dist -->

Commit message: gps yaw fix

File: description/rover_model/urdf/stand_link.urdf.xacro (robot description, xacro)
@@ -130,5 +130,5 @@
     </link>
     <joint name="imu_joint" type="fixed">
-        <origin xyz="0.159347 0 0" rpy="0 0 0" />
+        <origin xyz="0.159347 0 0" rpy="3.14159 0 0" />
         <!-- The x-pos is same as it's actual position on the stand, but z-pos same as base_link
              x: imu_x_dist_to_stand + chassis_to_stand_link_x_dist -->

Commit message: reverting the direction

File: description/rover_model/urdf/stand_link.urdf.xacro (robot description, xacro)
@@ -101,5 +101,5 @@
     <link name="imu_link">
         <inertial>
-            <origin xyz="3.0642E-07 -2.658E-07 0.0062442" rpy="0 0 0" />
+            <origin xyz="3.0642E-07 -2.658E-07 0.0062442" rpy="3.14159 0 0" />
             <mass value="0.016518" />
             <inertia
@@ -112,5 +112,5 @@
         </inertial>
         <visual>
-            <origin xyz="0 0 0" rpy="0 0 0" /> <!-- mesh origin matches FLU imu_link frame -->
+            <origin xyz="0 0 0" rpy="3.14159 0 0" /> <!-- Physical imu located on stand -->
             <!-- z-pos of visual model moved back up to stand height
                  z: imu_z_dist_to_stand + chassis_to_stand_link_z_dist + chassis_to_base_link_dist} -->
@@ -123,5 +123,5 @@
         </visual>
         <collision>
-            <origin xyz="0 0 0" rpy="0 0 0" />
+            <origin xyz="0 0 0" rpy="3.14159 0 0" />
             <geometry>
                 <mesh filename="package://description/rover_model/meshes/imu_link.STL" />
@@ -130,10 +130,9 @@
     </link>
     <joint name="imu_joint" type="fixed">
-        <!-- imu_link is FLU (x-forward, y-left, z-up), aligned with base_link.
-             ⚠ This rpy MUST match the PHYSICAL sensor axes. It is only valid if the
-             IMU is physically mounted FLU. If the chip is mounted flipped, TF will
-             rotate gyro/accel 180° about X (inverting roll/pitch and FLIPPING yaw
-             sign in ekf_local). Verify on the bench (see notes) before trusting. -->
-        <origin xyz="0.0969 0.0229 0" rpy="0 0 0" />
+        <!-- The IMU is physically mounted Z-DOWN (upside down), so imu_link is
+             rolled 180° about X relative to base_link. This rpy MUST match the
+             real sensor mounting — TF uses it to rotate gyro/accel into base_link.
+             If you ever remount the IMU FLU (x-fwd, y-left, z-up), change to "0 0 0". -->
+        <origin xyz="0.0969 0.0229 0" rpy="3.14159 0 0" />
         <!-- The x-pos is same as it's actual position on the stand, but z-pos same as base_link
              x: imu_x_dist_to_stand + chassis_to_stand_link_x_dist -->

Commit message: fix

File: description/rover_model/urdf/stand_link.urdf.xacro (robot description, xacro)
@@ -101,5 +101,5 @@
     <link name="imu_link">
         <inertial>
-            <origin xyz="3.0642E-07 -2.658E-07 0.0062442" rpy="3.14159 0 0" />
+            <origin xyz="3.0642E-07 -2.658E-07 0.0062442" rpy="0 0 0" />
             <mass value="0.016518" />
             <inertia
@@ -112,5 +112,5 @@
         </inertial>
         <visual>
-            <origin xyz="0 0 0" rpy="3.14159 0 0" /> <!-- Physical imu located on stand -->
+            <origin xyz="0 0 0" rpy="0 0 0" /> <!-- Physical imu located on stand -->
             <!-- z-pos of visual model moved back up to stand height
                  z: imu_z_dist_to_stand + chassis_to_stand_link_z_dist + chassis_to_base_link_dist} -->
@@ -123,5 +123,5 @@
         </visual>
         <collision>
-            <origin xyz="0 0 0" rpy="3.14159 0 0" />
+            <origin xyz="0 0 0" rpy="0 0 0" />
             <geometry>
                 <mesh filename="package://description/rover_model/meshes/imu_link.STL" />
@@ -134,5 +134,5 @@
              real sensor mounting — TF uses it to rotate gyro/accel into base_link.
              If you ever remount the IMU FLU (x-fwd, y-left, z-up), change to "0 0 0". -->
-        <origin xyz="0.0969 0.0229 0" rpy="3.14159 0 0" />
+        <origin xyz="0.0969 0.0229 0" rpy="0 0 0" />
         <!-- The x-pos is same as it's actual position on the stand, but z-pos same as base_link
              x: imu_x_dist_to_stand + chassis_to_stand_link_x_dist -->

Commit message: fixed sign error in URDF

File: description/rover_model/urdf/stand_link.urdf.xacro (robot description, xacro)
@@ -35,5 +35,5 @@
     </link>
     <joint name="stand_joint" type="fixed">
-        <origin xyz="0.1268 0 0.6548" rpy="0 0 0" />
+        <origin xyz="-0.1268 0 0.6548" rpy="0 0 0" />
         <parent link="chassis_link" />
         <child link="stand_link" />

Commit message: relay workoing, need to test for the offset parameter tuning.

File: description/rover_model/urdf/stand_link.urdf.xacro (robot description, xacro)
@@ -130,5 +130,5 @@
     </link>
     <joint name="imu_joint" type="fixed">
-        <origin xyz="0.159347 0 0" rpy="3.14159 0 0" />
+        <origin xyz="0.159347 0 0" rpy="0 0 0" />
         <!-- The x-pos is same as it's actual position on the stand, but z-pos same as base_link
              x: imu_x_dist_to_stand + chassis_to_stand_link_x_dist -->
