Commit message: fixed gazebo launch, robot spawn, odom launch, tf tree, reduced gazebo overhead

File: description/rover_model/urdf/constants.xacro (robot description, xacro)
@@ -1,4 +1,4 @@
 <?xml version="1.0"?>
-<robot name="espresso_constants" xmlns:xacro="http://ros.org/wiki/xacro">
+<robot name="timbot_constants" xmlns:xacro="http://ros.org/wiki/xacro">
     <!-- Drivebase -->
     <!-- <xacro:property name="base_length" value="1.268"/>
@@ -28,11 +28,11 @@
     <xacro:property name="wheels_separation" value="0.823976"/>
     <xacro:property name="wheel_diameter" value="0.25"/>
-    <xacro:property name="wheel_acceleration" value="1.0"/>
-    <xacro:property name="wheel_torque" value="20"/>
+    <xacro:property name="wheel_acceleration" value="5.0"/>
+    <xacro:property name="wheel_torque" value="60"/>
     <xacro:property name="wheel_mass" value="3.533"/>
     <!-- Gazebo Motor -->
     <xacro:property name="diff_drive_update_rate" value="30.0"/>
-    <xacro:property name="diff_drive_commandTopic" value="cmd_vel"/>
-    <xacro:property name="diff_drive_odometryTopic" value="odom"/>
+    <xacro:property name="diff_drive_commandTopic" value="/cmd_vel"/>
+    <xacro:property name="diff_drive_odometryTopic" value="/odom"/>
     <xacro:property name="diff_drive_odometryFrame" value="odom"/>
     <xacro:property name="diff_drive_robotBaseFrame" value="base_link"/>
@@ -59,7 +59,7 @@
     <xacro:property name="laser_noise_mean" value="0.0"/>
     <xacro:property name="laser_noise_stddev" value="0.01/3"/>
-    <xacro:property name="bottom_laser_topicName" value="scan_lower"/>
+    <xacro:property name="bottom_laser_topicName" value="/scan_lower"/>
     <xacro:property name="bottom_laser_frameName" value="bottom_lidar_link"/>
-    <xacro:property name="top_laser_topicName" value="scan_upper"/>
+    <xacro:property name="top_laser_topicName" value="/scan_upper"/>
     <xacro:property name="top_laser_frameName" value="top_lidar_link"/>
     <xacro:property name="distance_to_second_lidar" value="0.14"/>
@@ -69,10 +69,10 @@
     <xacro:property name="ZED_camera_length" value="0.175"/>
     <xacro:property name="ZED_camera_width" value="0.03"/>
-    <xacro:property name="ZED_camera_length" value="0.175"/>
+    <!-- <xacro:property name="ZED_camera_length" value="0.175"/> -->
     <xacro:property name="ZED_stereo_offset" value="0.12"/>
     <xacro:property name="ZED_camera_pitch" value="${30 * pi/180}"/>
     <!--<xacro:property name="ZED_camera_pitch" value="${50 * pi/180}"/>-->
     <!-- ZED image height/width corresponds to image size for 60Hz refresh-->
-    <xacro:property name="ZED_image_refresh" value="60"/>
+    <xacro:property name="ZED_image_refresh" value="0"/>
     <xacro:property name="ZED_image_width" value="640"/>
     <xacro:property name="ZED_image_height" value="360"/>
@@ -80,11 +80,11 @@
     <xacro:property name="ZED_image_hfov" value="${90 * pi/180}"/>
     <xacro:property name="ZED_name" value="zed_node"/>
-    <xacro:property name="ZED_always_on" value="true"/>
+    <xacro:property name="ZED_always_on" value="false"/>
     <xacro:property name="ZED_update_rate" value="0"/>
-    <xacro:property name="ZED_image_topicName" value="image_raw_color"/>
-    <xacro:property name="ZED_image_info_topicName" value="camera_info"/>
-    <xacro:property name="ZED_depth_topicName" value="depth/image_raw"/>
-    <xacro:property name="ZED_depth_info_topicName" value="depth/camera_info"/>
-    <xacro:property name="ZED_depth_points_topicName" value="depth/points"/>
+    <xacro:property name="ZED_image_topicName" value="/image_raw_color"/>
+    <xacro:property name="ZED_image_info_topicName" value="/camera_info"/>
+    <xacro:property name="ZED_depth_topicName" value="/depth/image_raw"/>
+    <xacro:property name="ZED_depth_info_topicName" value="/depth/camera_info"/>
+    <xacro:property name="ZED_depth_points_topicName" value="/depth/points"/>
     <xacro:property name="ZED_frameName" value="left_camera_link_optical"/>
     <!--ZED CAMERA JOINT PARAMETERS-->
@@ -94,6 +94,6 @@
     <!-- NOTE: approx. as a cylinder, Garmin itself is similar to a hockey puck -->
     <xacro:property name="gps_frame" value="gps_link"/>
-    <xacro:property name="gps_topic" value="gps/fix"/>
-    <xacro:property name="gps_vel_topic" value="gps/fix_velocity"/>
+    <xacro:property name="gps_topic" value="/gps/fix"/>
+    <xacro:property name="gps_vel_topic" value="/gps/fix_velocity"/>
     <xacro:property name="gps_update_rate" value="5.0"/>
     <!-- NOTE: GPS coordinates for UofT St. George Campus -->
@@ -105,5 +105,5 @@
     <!-- Phidget IMU -->
     <xacro:property name="imu_frame" value="imu_link"/>
-    <xacro:property name="imu_topic" value="imu/data"/>
+    <xacro:property name="imu_topic" value="/imu/data"/>
     <xacro:property name="imu_update_rate" value="128.0"/>
     <xacro:property name="imu_x_dist_to_stand" value="-0.018653"/>

File: description/rover_model/urdf/plugins.ignition.xacro (robot description, xacro)
@@ -31,7 +31,7 @@
             <min_angular_acceleration>-2.0</min_angular_acceleration>
             <odom_publish_frequency>30</odom_publish_frequency>
-            <topic>cmd_vel</topic>
-            <odom_topic>odom</odom_topic>
-            <tf_topic>tf</tf_topic>
+            <topic>/cmd_vel</topic>
+            <odom_topic>/odom</odom_topic>
+            <tf_topic>/tf</tf_topic>
             <frame_id>odom</frame_id>
             <child_frame_id>base_link</child_frame_id>
@@ -43,5 +43,5 @@
             <joint_name>${wheel_left_joint}</joint_name>
             <joint_name>${wheel_right_joint}</joint_name>
-            <topic>joint_states</topic>
+            <topic>/joint_states</topic>
         </plugin>
     </gazebo>
@@ -52,5 +52,5 @@
             <update_rate>${imu_update_rate}</update_rate>
             <visualize>true</visualize>
-            <topic>imu/data</topic>
+            <topic>/imu/data</topic>
             <ignition_frame_id>imu_link</ignition_frame_id>
             <enable_metrics>true</enable_metrics>
@@ -104,5 +104,5 @@
             <always_on>true</always_on>
             <update_rate>${gps_update_rate}</update_rate>
-            <topic>gps/fix</topic>
+            <topic>/gps/fix</topic>
             <navsat>
                 <position_sensing>
@@ -143,5 +143,5 @@
             <update_rate>${laser_update_rate}</update_rate>
             <visualize>${laser_visualize}</visualize>
-            <topic>scan_lower</topic>
+            <topic>/scan_lower</topic>
             <ignition_frame_id>bottom_lidar_link</ignition_frame_id>
             <lidar>
@@ -179,5 +179,5 @@
             <update_rate>${laser_update_rate}</update_rate>
             <visualize>${laser_visualize}</visualize>
-            <topic>scan_upper</topic>
+            <topic>/scan_upper</topic>
             <ignition_frame_id>top_lidar_link</ignition_frame_id>
             <lidar>
@@ -215,5 +215,5 @@
             <update_rate>${ZED_image_refresh}</update_rate>
             <visualize>false</visualize>
-            <topic>zed_node/left/image_raw</topic>
+            <topic>/zed_node/left/image_raw</topic>
             <camera>
                 <horizontal_fov>${ZED_image_hfov}</horizontal_fov>

File: description/rover_model/urdf/timbot.urdf.xacro (robot description, xacro)
@@ -3,5 +3,5 @@
      Commit Version: 1.6.0-4-g7f85cfe  Build Version: 1.6.7995.38578
      For more information, please see http://wiki.ros.org/sw_urdf_exporter -->
-<robot name="espresso" xmlns:xacro="http://ros.org/wiki/xacro">
+<robot name="timbot" xmlns:xacro="http://ros.org/wiki/xacro">
 	<!-- Argument to select Gazebo version: 'classic' or 'ignition' -->
 	<xacro:arg name="gazebo_version" default="ignition"/>
@@ -39,8 +39,14 @@
 			</material>
 		</visual>
+		<!-- <collision>
+			<origin xyz="0 0 0" rpy="0 0 0" />
+			<geometry>
+				<mesh filename="package://description/rover_model/meshes/chassis_link.STL" />
+			</geometry>
+		</collision> -->
 		<collision>
 			<origin xyz="0 0 0" rpy="0 0 0" />
 			<geometry>
-				<mesh filename="package://description/rover_model/meshes/chassis_link.STL" />
+				<box size="0.9 0.6 0.3"/>
 			</geometry>
 		</collision>

File: description/rover_model/urdf/wheels.urdf.xacro (robot description, xacro)
@@ -36,8 +36,13 @@
             </material>
         </visual>
-        <collision>
+        <!-- <collision>
             <origin xyz="0 0 0" rpy="0 0 0" />
             <geometry>
                 <mesh filename="package://description/rover_model/meshes/leftwheel_link.STL" />
+            </geometry>
+        </collision> -->
+        <collision>
+            <origin xyz="0 0 0" rpy="1.5707 0 0" /> <geometry>
+                <cylinder length="0.1" radius="0.125"/>
             </geometry>
         </collision>
@@ -48,4 +53,5 @@
         <child link="left_wheel_link" />
         <axis xyz="0 1 0" />
+        <limit effort="100.0" velocity="20.0"/>
     </joint>
     <gazebo reference="left_wheel_link">
@@ -79,8 +85,13 @@
             </material>
         </visual>
-        <collision>
+        <!-- <collision>
             <origin xyz="0 0 0" rpy="0 0 0" />
             <geometry>
                 <mesh filename="package://description/rover_model/meshes/rightwheel_link.STL" />
+            </geometry>
+        </collision> -->
+        <collision>
+            <origin xyz="0 0 0" rpy="1.5707 0 0" /> <geometry>
+                <cylinder length="0.1" radius="0.125"/>
             </geometry>
         </collision>
@@ -91,4 +102,5 @@
         <child link="right_wheel_link" />
         <axis xyz="0 1 0" />
+        <limit effort="100.0" velocity="20.0"/>
     </joint>
     <gazebo reference="right_wheel_link">

Commit message: added cv support in sim

File: description/rover_model/urdf/constants.xacro (robot description, xacro)
@@ -71,15 +71,15 @@
     <!-- <xacro:property name="ZED_camera_length" value="0.175"/> -->
     <xacro:property name="ZED_stereo_offset" value="0.12"/>
-    <xacro:property name="ZED_camera_pitch" value="${30 * pi/180}"/>
+    <xacro:property name="ZED_camera_pitch" value="${25 * pi/180}"/>
     <!--<xacro:property name="ZED_camera_pitch" value="${50 * pi/180}"/>-->
     <!-- ZED image height/width corresponds to image size for 60Hz refresh-->
-    <xacro:property name="ZED_image_refresh" value="0"/>
-    <xacro:property name="ZED_image_width" value="640"/>
-    <xacro:property name="ZED_image_height" value="360"/>
+    <xacro:property name="ZED_image_refresh" value="5"/>
+    <xacro:property name="ZED_image_width" value="320"/>
+    <xacro:property name="ZED_image_height" value="180"/>
     <xacro:property name="ZED_image_format" value="R8G8B8"/>
-    <xacro:property name="ZED_image_hfov" value="${90 * pi/180}"/>
+    <xacro:property name="ZED_image_hfov" value="${110 * pi/180}"/>
     <xacro:property name="ZED_name" value="zed_node"/>
-    <xacro:property name="ZED_always_on" value="false"/>
-    <xacro:property name="ZED_update_rate" value="0"/>
+    <xacro:property name="ZED_always_on" value="true"/>
+    <xacro:property name="ZED_update_rate" value="5"/>
     <xacro:property name="ZED_image_topicName" value="/image_raw_color"/>
     <xacro:property name="ZED_image_info_topicName" value="/camera_info"/>

File: description/rover_model/urdf/plugins.ignition.xacro (robot description, xacro)
@@ -8,5 +8,5 @@
     <gazebo>
         <plugin filename="ignition-gazebo-sensors-system" name="ignition::gazebo::systems::Sensors">
-            <render_engine>ogre2</render_engine>
+            <render_engine>ogre</render_engine>
         </plugin>
     </gazebo>
@@ -210,22 +210,29 @@
         </sensor>
     </gazebo>
-    <!-- Stereo Camera (left) -->
+    <!-- Stereo Camera (left) — only included when enable_camera arg is true -->
+    <xacro:if value="$(arg enable_camera)">
     <gazebo reference="left_camera_link">
-        <sensor name="camera_left" type="camera">
-            <always_on>true</always_on>
-            <update_rate>${ZED_image_refresh}</update_rate>
+        <sensor name="camera_left" type="rgbd_camera">
+            <always_on>true</always_on>
+            <update_rate>$(arg camera_fps)</update_rate>
             <visualize>false</visualize>
-            <topic>/zed_node/left/image_raw</topic>
+            <topic>/zed_node/left</topic>
             <camera>
                 <horizontal_fov>${ZED_image_hfov}</horizontal_fov>
                 <image>
-                    <width>${ZED_image_width}</width>
-                    <height>${ZED_image_height}</height>
+                    <width>$(arg camera_width)</width>
+                    <height>$(arg camera_height)</height>
                     <format>R8G8B8</format>
                 </image>
                 <clip>
-                    <near>0.02</near>
+                    <near>0.3</near>
                     <far>300</far>
                 </clip>
+                <depth_camera>
+                    <clip>
+                        <near>0.3</near>
+                        <far>10</far>
+                    </clip>
+                </depth_camera>
                 <noise>
                     <type>gaussian</type>
@@ -236,3 +243,4 @@
         </sensor>
     </gazebo>
+    </xacro:if>
 </robot>

File: description/rover_model/urdf/timbot.urdf.xacro (robot description, xacro)
@@ -6,4 +6,10 @@
 	<!-- Argument to select Gazebo version: 'classic' or 'ignition' -->
 	<xacro:arg name="gazebo_version" default="ignition"/>
+	<!-- Argument to enable/disable the ZED camera sensor in simulation -->
+	<xacro:arg name="enable_camera" default="false"/>
+	<!-- Camera settings (only used when enable_camera is true) -->
+	<xacro:arg name="camera_fps" default="5"/>
+	<xacro:arg name="camera_width" default="320"/>
+	<xacro:arg name="camera_height" default="180"/>
 	<link name="base_link" />
 	<!-- Includes - Select plugins based on Gazebo version -->

Commit message: updating camera and adding relay to depth map

File: description/rover_model/urdf/constants.xacro (robot description, xacro)
@@ -71,5 +71,5 @@
     <!-- <xacro:property name="ZED_camera_length" value="0.175"/> -->
     <xacro:property name="ZED_stereo_offset" value="0.12"/>
-    <xacro:property name="ZED_camera_pitch" value="${25 * pi/180}"/>
+    <xacro:property name="ZED_camera_pitch" value="${20 * pi/180}"/>
     <!--<xacro:property name="ZED_camera_pitch" value="${50 * pi/180}"/>-->
     <!-- ZED image height/width corresponds to image size for 60Hz refresh-->

Commit message: developed new odom pathway. Still need to test with wheel encoders, and test with the gps to see cartographer performance. Changed wheel encoder topic to wheel_odom

File: description/rover_model/urdf/constants.xacro (robot description, xacro)
@@ -34,5 +34,5 @@
     <xacro:property name="diff_drive_update_rate" value="30.0"/>
     <xacro:property name="diff_drive_commandTopic" value="/cmd_vel"/>
-    <xacro:property name="diff_drive_odometryTopic" value="/odom"/>
+    <xacro:property name="diff_drive_odometryTopic" value="/wheel_odom"/>
     <xacro:property name="diff_drive_odometryFrame" value="odom"/>
     <xacro:property name="diff_drive_robotBaseFrame" value="base_link"/>

Commit message: finally fucking did it

File: description/rover_model/urdf/constants.xacro (robot description, xacro)
@@ -26,5 +26,5 @@
     <xacro:property name="wheel_left_joint" value="left_wheel_joint"/>
     <xacro:property name="wheel_right_joint" value="right_wheel_joint"/>
-    <xacro:property name="wheels_separation" value="0.823976"/>
+    <xacro:property name="wheels_separation" value="0.6744"/>
     <xacro:property name="wheel_diameter" value="0.25"/>
     <xacro:property name="wheel_acceleration" value="5.0"/>
@@ -71,5 +71,5 @@
     <!-- <xacro:property name="ZED_camera_length" value="0.175"/> -->
     <xacro:property name="ZED_stereo_offset" value="0.12"/>
-    <xacro:property name="ZED_camera_pitch" value="${20 * pi/180}"/>
+    <xacro:property name="ZED_camera_pitch" value="${12 * pi/180}"/>
     <!--<xacro:property name="ZED_camera_pitch" value="${50 * pi/180}"/>-->
     <!-- ZED image height/width corresponds to image size for 60Hz refresh-->

File: description/rover_model/urdf/stand_link.urdf.xacro (robot description, xacro)
@@ -35,5 +35,5 @@
     </link>
     <joint name="stand_joint" type="fixed">
-        <origin xyz="0.178 0.001524 0.26861" rpy="0 0 0" />
+        <origin xyz="0.1268 0 0.6548" rpy="0 0 0" />
         <parent link="chassis_link" />
         <child link="stand_link" />
@@ -74,5 +74,5 @@
     </link>
     <joint name="zed_joint" type="fixed">
-        <origin xyz="0.044163 0 ${ZED_camera_to_top_plate_z}" rpy="0 ${ZED_camera_pitch} 0" />
+        <origin xyz="0.0736 0 0.102" rpy="0 ${ZED_camera_pitch} 0" />
         <parent link="stand_link" />
         <child link="zed_link" />
@@ -101,5 +101,5 @@
     <link name="imu_link">
         <inertial>
-            <origin xyz="3.0642E-07 -2.658E-07 0.0062442" rpy="0 0 0" />
+            <origin xyz="3.0642E-07 -2.658E-07 0.0062442" rpy="3.14159 0 0" />
             <mass value="0.016518" />
             <inertia
@@ -112,5 +112,5 @@
         </inertial>
         <visual>
-            <origin xyz="0 0 0" rpy="0 0 0" /> <!-- Physical imu located on stand -->
+            <origin xyz="0 0 0" rpy="3.14159 0 0" /> <!-- Physical imu located on stand -->
             <!-- z-pos of visual model moved back up to stand height
                  z: imu_z_dist_to_stand + chassis_to_stand_link_z_dist + chassis_to_base_link_dist} -->
@@ -123,5 +123,5 @@
         </visual>
         <collision>
-            <origin xyz="0 0 0" rpy="0 0 0" />
+            <origin xyz="0 0 0" rpy="3.14159 0 0" />
             <geometry>
                 <mesh filename="package://description/rover_model/meshes/imu_link.STL" />
@@ -130,5 +130,5 @@
     </link>
     <joint name="imu_joint" type="fixed">
-        <origin xyz="0.159347 0 0" rpy="0 0 0" />
+        <origin xyz="0.0969 0.0229 0" rpy="3.14159 0 0" />
         <!-- The x-pos is same as it's actual position on the stand, but z-pos same as base_link
              x: imu_x_dist_to_stand + chassis_to_stand_link_x_dist -->
@@ -170,5 +170,5 @@
     </link>
     <joint name="gps_joint" type="fixed">
-        <origin xyz="-0.054799 0 0.0095015" rpy="0 0 0" />
+        <origin xyz="-0.0288 0.0274 0.0095015" rpy="0 0 0" />
         <parent link="stand_link" />
         <child link="gps_link" />

File: description/rover_model/urdf/timbot.urdf.xacro (robot description, xacro)
@@ -26,5 +26,5 @@
 	<link name="chassis_link">
 		<inertial>
-			<origin xyz="-0.040859 0.00033673 -0.054592" rpy="0 0 0" />
+			<origin xyz="-0.040859 0.00033673 10.54592" rpy="0 0 0" />
 			<mass value="40.135" />
 			<inertia
@@ -59,5 +59,5 @@
 	</link>
 	<joint name="chassis_joint" type="fixed">
-		<origin xyz="0 0 0.34041" rpy="0 0 0" />
+		<origin xyz="0.2573 0 0.1301" rpy="0 0 0" />
 		<parent link="base_link" />
 		<child link="chassis_link" />
@@ -97,5 +97,5 @@
 	</link>
 	<joint name="top_lidar_joint" type="fixed">
-		<origin xyz="0.52049 -0.005698 ${distance_to_second_lidar - 0.069334}" rpy="0 0 0" />
+		<origin xyz="0.2092 0.0005 0.3470" rpy="0 0 0" />
 		<!-- before z =  0.0056661 -->
 		<parent link="chassis_link" />
@@ -136,5 +136,5 @@
 	</link>
 	<joint name="bottom_lidar_joint" type="fixed">
-		<origin xyz="0.52049 -0.005698 -0.069334" rpy="0 0 0" />
+		<origin xyz="0.2535 0 0.1438" rpy="0 0 0" />
 		<parent link="chassis_link" />
 		<child link="bottom_lidar_link" />

File: description/rover_model/urdf/wheels.urdf.xacro (robot description, xacro)
@@ -49,5 +49,5 @@
     </link>
     <joint name="left_wheel_joint" type="continuous">
-        <origin xyz="0.30478 0.40518 -0.21541" rpy="0 0 0" />
+        <origin xyz="0 0.3372 0" rpy="0 0 0" />
         <parent link="chassis_link" />
         <child link="left_wheel_link" />
@@ -98,5 +98,5 @@
     </link>
     <joint name="right_wheel_joint" type="continuous">
-        <origin xyz="0.30482 -0.40518 -0.21541" rpy="0 0 0" />
+        <origin xyz="0 -0.3372 0" rpy="0 0 0" />
         <parent link="chassis_link" />
         <child link="right_wheel_link" />
@@ -142,5 +142,5 @@
     </link>
     <joint name="caster_joint" type="fixed">
-        <origin xyz="-0.36833 0.001524 -0.13183" rpy="0 0 0" />
+        <origin xyz="-0.6730 0 0.0702" rpy="0 0 0" />
         <parent link="chassis_link" />
         <child link="caster_link" />

Commit message: working relay + working nav node + fixed zed tf

File: description/rover_model/urdf/constants.xacro (robot description, xacro)
@@ -71,5 +71,5 @@
     <!-- <xacro:property name="ZED_camera_length" value="0.175"/> -->
     <xacro:property name="ZED_stereo_offset" value="0.12"/>
-    <xacro:property name="ZED_camera_pitch" value="${12 * pi/180}"/>
+    <xacro:property name="ZED_camera_pitch" value="${27 * pi/180}"/>
     <!--<xacro:property name="ZED_camera_pitch" value="${50 * pi/180}"/>-->
     <!-- ZED image height/width corresponds to image size for 60Hz refresh-->

File: description/rover_model/urdf/stand_link.urdf.xacro (robot description, xacro)
@@ -74,5 +74,5 @@
     </link>
     <joint name="zed_joint" type="fixed">
-        <origin xyz="0.0736 0 0.102" rpy="0 ${ZED_camera_pitch} 0" />
+        <origin xyz="0.0736 0 0.06" rpy="0 ${ZED_camera_pitch} 0" />
         <parent link="stand_link" />
         <child link="zed_link" />
